Commit message: Add effort limit to robot joints

File: kuka_kr150_support/urdf/kr150r3100_2_macro.xacro (robot description, xacro)
@@ -132,5 +132,5 @@
       <child link="${prefix}link_1"/>
       <axis xyz="0 0 -1"/>
-      <limit effort="0" lower="${radians(-185)}" upper="${radians(185)}" velocity="${radians(105)}"/>
+      <limit effort="1000" lower="${radians(-185)}" upper="${radians(185)}" velocity="${radians(105)}"/>
     </joint>
     <!-- joint 2 (A2) -->
@@ -140,5 +140,5 @@
       <child link="${prefix}link_2"/>
       <axis xyz="0 1 0"/>
-      <limit effort="0" lower="${radians(-140)}" upper="${radians(-5)}" velocity="${radians(107)}"/>
+      <limit effort="1000" lower="${radians(-140)}" upper="${radians(-5)}" velocity="${radians(107)}"/>
     </joint>
     <!-- joint 3 (A3) -->
@@ -148,5 +148,5 @@
       <child link="${prefix}link_3"/>
       <axis xyz="0 1 0"/>
-      <limit effort="0" lower="${radians(-120)}" upper="${radians(168)}" velocity="${radians(114)}"/>
+      <limit effort="1000" lower="${radians(-120)}" upper="${radians(168)}" velocity="${radians(114)}"/>
     </joint>
     <!-- joint 4 (A4) -->
@@ -156,5 +156,5 @@
       <child link="${prefix}link_4"/>
       <axis xyz="-1 0 0"/>
-      <limit effort="0" lower="${radians(-350)}" upper="${radians(350)}" velocity="${radians(190)}"/>
+      <limit effort="1000" lower="${radians(-350)}" upper="${radians(350)}" velocity="${radians(190)}"/>
     </joint>
     <!-- joint 5 (A5) -->
@@ -164,5 +164,5 @@
       <child link="${prefix}link_5"/>
       <axis xyz="0 1 0"/>
-      <limit effort="0" lower="${radians(-125)}" upper="${radians(125)}" velocity="${radians(180)}"/>
+      <limit effort="1000" lower="${radians(-125)}" upper="${radians(125)}" velocity="${radians(180)}"/>
     </joint>
     <!-- joint 6 (A6) -->
@@ -172,5 +172,5 @@
       <child link="${prefix}link_6"/>
       <axis xyz="-1 0 0"/>
-      <limit effort="0" lower="${radians(-350)}" upper="${radians(350)}" velocity="${radians(260)}"/>
+      <limit effort="1000" lower="${radians(-350)}" upper="${radians(350)}" velocity="${radians(260)}"/>
     </joint>
     <!-- ROS-Industrial 'base' frame - base_link to KUKA $ROBROOT coordinate system transform -->
